File: hardware/Meow Meow.sch (KiCad schematic (older format))
At the start: 27 parts, among them P1 D, P10 A, P11 W, P12 MOUSE_LEFT, P13 CONN_01X12, P2 SPACE, P3 KEY_RIGHT_ARROW, P4 CONN_02X03, P5 KEY_LEFT_ARROW, P6 KEY_DOWN_ARROW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

Commit message: Change Headers Expansion and SWD
Parts:
- removed P13: CONN_01X12, Pin_Headers:Pin_Header_Straight_1x12_Pitch2.54mm, symbol CONN_01X12
- removed P4: CONN_02X03, Pin_Headers:Pin_Header_Straight_2x03_Pitch2.54mm, symbol CONN_02X03
- added P13: Expansion, Pines:610X1221121, symbol CONN_02X06
- added P4: SWD, Pines:61000418321, symbol CONN_01X04
- P1, P10, P11, P12, P2, P3, P5, P6, P7, P8: footprint MeowMeow:ALLIGATORCLIP -> Connectors:SEWALLI
Connections:
- net labels removed: RESET
- wire segments 98 -> 97
- no-connect marks 15 -> 14
Changed lines of the file:
@@
 Title "Meow Meow"
 Date "2018-05-16"
-Rev "0.4"
+Rev "0.6"
 Comp "Electronic Cats"
 Comment1 "Andres Sabas"
@@
 F 0 "P7" H 10435 5070 60  0000 C CNN
 F 1 "KEY_UP_ARROW" H 10435 4870 60  0000 C CNN
-F 2 "MeowMeow:ALLIGATORCLIP" H 10435 4970 60  0001 C CNN
+F 2 "Connectors:SEWALLI" H 10435 4970 60  0001 C CNN
 F 3 "" H 10435 4970 60  0001 C CNN
 	1    10435 4970
@@
 F 0 "P6" H 10125 5095 60  0000 C CNN
 F 1 "KEY_DOWN_ARROW" H 10125 4895 60  0000 C CNN
-F 2 "MeowMeow:ALLIGATORCLIP" H 10125 4995 60  0001 C CNN
+F 2 "Connectors:SEWALLI" H 10125 4995 60  0001 C CNN
 F 3 "" H 10125 4995 60  0001 C CNN
 	1    10125 4995
@@
 F 0 "P3" H 9470 5100 60  0000 C CNN
 F 1 "KEY_RIGHT_ARROW" H 9470 4900 60  0000 C CNN
-F 2 "MeowMeow:ALLIGATORCLIP" H 9470 5000 60  0001 C CNN
+F 2 "Connectors:SEWALLI" H 9470 5000 60  0001 C CNN
 F 3 "" H 9470 5000 60  0001 C CNN
 	1    9470 5000
@@
 F 0 "P2" H 9160 5100 60  0000 C CNN
 F 1 "SPACE" H 9160 4900 60  0000 C CNN
-F 2 "MeowMeow:ALLIGATORCLIP" H 9160 5000 60  0001 C CNN
+F 2 "Connectors:SEWALLI" H 9160 5000 60  0001 C CNN
 F 3 "" H 9160 5000 60  0001 C CNN
 	1    9160 5000
@@
 Text Label 10790 3515 0    60   ~ 0
 D8
-$Comp
-L CONN_02X03 P4
-U 1 1 5AD9B33E
-P 8955 3335
-F 0 "P4" H 8955 3535 50  0000 C CNN
-F 1 "CONN_02X03" H 8955 3135 50  0000 C CNN
-F 2 "Pin_Headers:Pin_Header_Straight_2x03_Pitch2.54mm" H 8955 2135 50  0001 C CNN
-F 3 "" H 8955 2135 50  0000 C CNN
-	1    8955 3335
-	1    0    0    -1
-$EndComp
-Text Label 9330 3435 0    60   ~ 0
-RESET
-Text Label 8560 3235 2    60   ~ 0
+Text Label 8970 3285 2    60   ~ 0
 SWDIO
-Text Label 8560 3435 2    60   ~ 0
+Text Label 8975 3385 2    60   ~ 0
 SWCLK
 $Comp
 L +3.3V #PWR06
 U 1 1 5AD9BCA9
-P 9660 3300
-F 0 "#PWR06" H 9660 3150 50  0001 C CNN
-F 1 "+3.3V" H 9660 3440 50  0000 C CNN
-F 2 "" H 9660 3300 50  0000 C CNN
-F 3 "" H 9660 3300 50  0000 C CNN
-	1    9660 3300
+P 8745 3570
+F 0 "#PWR06" H 8745 3420 50  0001 C CNN
+F 1 "+3.3V" H 8745 3710 50  0000 C CNN
+F 2 "" H 8745 3570 50  0000 C CNN
+F 3 "" H 8745 3570 50  0000 C CNN
+	1    8745 3570
 	1    0    0    -1
 $EndComp
@@
 L GND #PWR07
 U 1 1 5AD9BD50
-P 9330 3235
-F 0 "#PWR07" H 9330 2985 50  0001 C CNN
-F 1 "GND" H 9330 3085 50  0000 C CNN
-F 2 "" H 9330 3235 50  0000 C CNN
-F 3 "" H 9330 3235 50  0000 C CNN
-	1    9330 3235
-	0    -1   -1   0
-$EndComp
-NoConn ~ 8705 3335
+P 8985 3585
+F 0 "#PWR07" H 8985 3335 50  0001 C CNN
+F 1 "GND" H 8990 3435 50  0000 C CNN
+F 2 "" H 8985 3585 50  0000 C CNN
+F 3 "" H 8985 3585 50  0000 C CNN
+	1    8985 3585
+	1    0    0    -1
+$EndComp
 $Comp
 L R_Small R1
@@
 F 0 "P5" H 9810 5100 60  0000 C CNN
 F 1 "KEY_LEFT_ARROW" H 9810 4900 60  0000 C CNN
-F 2 "MeowMeow:ALLIGATORCLIP" H 9810 5000 60  0001 C CNN
+F 2 "Connectors:SEWALLI" H 9810 5000 60  0001 C CNN
 F 3 "" H 9810 5000 60  0001 C CNN
 	1    9810 5000
@@
 F 0 "P12" H 8660 5045 60  0000 C CNN
 F 1 "MOUSE_LEFT" H 8660 4845 60  0000 C CNN
-F 2 "MeowMeow:ALLIGATORCLIP" H 8660 4945 60  0001 C CNN
+F 2 "Connectors:SEWALLI" H 8660 4945 60  0001 C CNN
 F 3 "" H 8660 4945 60  0001 C CNN
 	1    8660 4945
@@
 F 0 "P11" H 8380 5070 60  0000 C CNN
 F 1 "W" H 8380 4870 60  0000 C CNN
-F 2 "MeowMeow:ALLIGATORCLIP" H 8380 4970 60  0001 C CNN
+F 2 "Connectors:SEWALLI" H 8380 4970 60  0001 C CNN
 F 3 "" H 8380 4970 60  0001 C CNN
 	1    8380 4970
@@
 F 0 "P8" H 7740 5070 60  0000 C CNN
 F 1 "S" H 7740 4870 60  0000 C CNN
-F 2 "MeowMeow:ALLIGATORCLIP" H 7740 4970 60  0001 C CNN
+F 2 "Connectors:SEWALLI" H 7740 4970 60  0001 C CNN
 F 3 "" H 7740 4970 60  0001 C CNN
 	1    7740 4970
@@
 F 0 "P1" H 7355 5060 60  0000 C CNN
 F 1 "D" H 7355 4860 60  0000 C CNN
-F 2 "MeowMeow:ALLIGATORCLIP" H 7355 4960 60  0001 C CNN
+F 2 "Connectors:SEWALLI" H 7355 4960 60  0001 C CNN
 F 3 "" H 7355 4960 60  0001 C CNN
 	1    7355 4960
@@
 F 0 "P10" H 8065 5075 60  0000 C CNN
 F 1 "A" H 8065 4875 60  0000 C CNN
-F 2 "MeowMeow:ALLIGATORCLIP" H 8065 4975 60  0001 C CNN
+F 2 "Connectors:SEWALLI" H 8065 4975 60  0001 C CNN
 F 3 "" H 8065 4975 60  0001 C CNN
 	1    8065 4975
@@
 Text Notes 7805 5625 0    60   ~ 0
 PIN EXTRAS
+Text Label 9490 5760 0    60   ~ 0
+I2S_SCK
+Text Label 9495 5860 0    60   ~ 0
+I2S_D1/X7
+Text Label 9495 5960 0    60   ~ 0
+TX/X2
+Text Label 9495 6060 0    60   ~ 0
+RX/X3
+Text Label 8780 5760 2    60   ~ 0
+MOSI
+Text Label 8780 5860 2    60   ~ 0
+MISO
+Text Label 8780 5960 2    60   ~ 0
+SCK
+Text Label 9495 6160 0    60   ~ 0
+CS
+Text Label 8785 6060 2    60   ~ 0
+SDA
+Text Label 8785 6160 2    60   ~ 0
+SCL
+$Comp
+L GND #PWR019
+U 1 1 5AFF5159
+P 9510 6260
+F 0 "#PWR019" H 9510 6010 50  0001 C CNN
+F 1 "GND" H 9510 6110 50  0000 C CNN
+F 2 "" H 9510 6260 50  0000 C CNN
+F 3 "" H 9510 6260 50  0000 C CNN
+	1    9510 6260
+	1    0    0    -1
+$EndComp
+$Comp
+L +3.3V #PWR020
+U 1 1 5AFF522D
+P 8500 6260
+F 0 "#PWR020" H 8500 6110 50  0001 C CNN
+F 1 "+3.3V" H 8500 6400 50  0000 C CNN
+F 2 "" H 8500 6260 50  0000 C CNN
+F 3 "" H 8500 6260 50  0000 C CNN
+	1    8500 6260
+	1    0    0    -1
+$EndComp
+$Comp
+L SW_Push SW1
+U 1 1 5B071A82
+P 1835 1655
+F 0 "SW1" H 1885 1755 50  0000 L CNN
+F 1 "SW_Push" H 1835 1595 50  0000 C CNN
+F 2 "TIH:SW_B3U-1000P" H 1835 1855 50  0001 C CNN
+F 3 "" H 1835 1855 50  0000 C CNN
+	1    1835 1655
+	1    0    0    -1
+$EndComp
+$Comp
+L GND #PWR021
+U 1 1 5B0727F0
+P 1590 1675
+F 0 "#PWR021" H 1590 1425 50  0001 C CNN
+F 1 "GND" H 1590 1525 50  0000 C CNN
+F 2 "" H 1590 1675 50  0000 C CNN
+F 3 "" H 1590 1675 50  0000 C CNN
+	1    1590 1675
+	1    0    0    -1
+$EndComp
+$Comp
+L CONN_02X06 P13
+U 1 1 5B19929F
+P 9140 6010
+F 0 "P13" H 9140 6360 50  0000 C CNN
+F 1 "Expansion" H 9140 5660 50  0000 C CNN
+F 2 "Pines:610X1221121" H 9140 4810 50  0001 C CNN
+F 3 "" H 9140 4810 50  0000 C CNN
+	1    9140 6010
+	1    0    0    -1
+$EndComp
+$Comp
+L CONN_01X04 P4
+U 1 1 5B19B71A
+P 9300 3435
+F 0 "P4" H 9300 3685 50  0000 C CNN
+F 1 "SWD" V 9400 3435 50  0000 C CNN
+F 2 "Pines:61000418321" H 9300 3435 50  0001 C CNN
+F 3 "" H 9300 3435 50  0000 C CNN
+	1    9300 3435
+	1    0    0    -1
+$EndComp
 Wire Wire Line
 	2495 3855 2355 3855
@@
 Wire Wire Line
 	9810 5100 9810 5325
-Wire Wire Line
-	9660 3335 9660 3300
-Wire Wire Line
-	8705 3435 8560 3435
-Wire Wire Line
-	9660 3335 9660 3300
-Wire Wire Line
-	9330 3435 9205 3435
-Wire Wire Line
-	9205 3335 9660 3335
-Wire Wire Line
-	9330 3235 9205 3235
 Wire Wire Line
 	10710 3515 10790 3515
@@
 Wire Wire Line
 	2495 3055 2310 3055
-Wire Wire Line
-	9900 5920 9900 6025
-Wire Wire Line
-	9800 5920 9800 6025
-Wire Wire Line
-	9700 5920 9700 6025
-Wire Wire Line
-	9600 5920 9600 6025
-Wire Wire Line
-	9500 5920 9500 6025
-Wire Wire Line
-	9400 5920 9400 6025
-Wire Wire Line
-	9300 5920 9300 6020
-Wire Wire Line
-	9200 5920 9200 6025
-Wire Wire Line
-	9100 5920 9100 6025
-Wire Wire Line
-	9000 5920 9000 6025
-Text Label 9900 6025 3    60   ~ 0
-I2S_SCK
-Text Label 9800 6025 3    60   ~ 0
-I2S_D1/X7
-Text Label 9700 6025 3    60   ~ 0
-TX/X2
-Text Label 9600 6025 3    60   ~ 0
-RX/X3
-Text Label 9500 6025 3    60   ~ 0
-MOSI
-Text Label 9400 6025 3    60   ~ 0
-MISO
-Text Label 9300 6020 3    60   ~ 0
-SCK
-Text Label 9200 6025 3    60   ~ 0
-CS
-Text Label 9100 6025 3    60   ~ 0
-SDA
-Text Label 9000 6025 3    60   ~ 0
-SCL
-$Comp
-L CONN_01X12 P13
-U 1 1 5AFF4EA1
-P 9350 5720
-F 0 "P13" H 9350 6370 50  0000 C CNN
-F 1 "CONN_01X12" V 9450 5720 50  0000 C CNN
-F 2 "Pin_Headers:Pin_Header_Straight_1x12_Pitch2.54mm" H 9350 5720 50  0001 C CNN
-F 3 "" H 9350 5720 50  0000 C CNN
-	1    9350 5720
-	0    -1   -1   0
-$EndComp
-Wire Wire Line
-	8900 5920 8900 6145
-Wire Wire Line
-	8800 5920 8800 6070
-$Comp
-L GND #PWR019
-U 1 1 5AFF5159
-P 8900 6145
-F 0 "#PWR019" H 8900 5895 50  0001 C CNN
-F 1 "GND" H 8900 5995 50  0000 C CNN
-F 2 "" H 8900 6145 50  0000 C CNN
-F 3 "" H 8900 6145 50  0000 C CNN
-	1    8900 6145
-	1    0    0    -1
-$EndComp
-$Comp
-L +3.3V #PWR020
-U 1 1 5AFF522D
-P 8660 6060
-F 0 "#PWR020" H 8660 5910 50  0001 C CNN
-F 1 "+3.3V" H 8660 6200 50  0000 C CNN
-F 2 "" H 8660 6060 50  0000 C CNN
-F 3 "" H 8660 6060 50  0000 C CNN
-	1    8660 6060
-	1    0    0    -1
-$EndComp
-Wire Wire Line
-	8660 6060 8660 6070
-Wire Wire Line
-	8660 6070 8800 6070
 Wire Notes Line
 	6970 5515 11215 5515
 Wire Notes Line
 	11215 5515 11215 5520
-$Comp
-L SW_Push SW1
-U 1 1 5B071A82
-P 1835 1655
-F 0 "SW1" H 1885 1755 50  0000 L CNN
-F 1 "SW_Push" H 1835 1595 50  0000 C CNN
-F 2 "TIH:SW_B3U-1000P" H 1835 1855 50  0001 C CNN
-F 3 "" H 1835 1855 50  0000 C CNN
-	1    1835 1655
-	1    0    0    -1
-$EndComp
 Wire Wire Line
 	2115 1655 2035 1655
@@
 Wire Wire Line
 	1590 1655 1590 1675
-$Comp
-L GND #PWR021
-U 1 1 5B0727F0
-P 1590 1675
-F 0 "#PWR021" H 1590 1425 50  0001 C CNN
-F 1 "GND" H 1590 1525 50  0000 C CNN
-F 2 "" H 1590 1675 50  0000 C CNN
-F 3 "" H 1590 1675 50  0000 C CNN
-	1    1590 1675
-	1    0    0    -1
-$EndComp
+Wire Wire Line
+	8890 6160 8785 6160
+Wire Wire Line
+	8890 6060 8785 6060
+Wire Wire Line
+	8890 5960 8780 5960
+Wire Wire Line
+	8890 5860 8780 5860
+Wire Wire Line
+	8890 5760 8780 5760
+Wire Wire Line
+	9390 6160 9495 6160
+Wire Wire Line
+	9390 6060 9495 6060
+Wire Wire Line
+	9390 5960 9495 5960
+Wire Wire Line
+	9390 5860 9495 5860
+Wire Wire Line
+	9390 5760 9490 5760
+Wire Wire Line
+	8500 6260 8890 6260
+Wire Wire Line
+	9390 6260 9510 6260
+Wire Wire Line
+	9100 3285 8970 3285
+Wire Wire Line
+	9100 3385 8975 3385
+Wire Wire Line
+	8830 3485 9100 3485
+Wire Wire Line
+	9100 3585 8985 3585
+Wire Wire Line
+	8830 3485 8830 3600
+Wire Wire Line
+	8830 3600 8745 3600
+Wire Wire Line
+	8745 3600 8745 3570
 $EndSCHEMATC

Commit message: added new connector
Parts:
- P1, P10, P11, P12, P2, P3, P5, P6, P7, P8: footprint Connectors:SEWALLI -> Connectors_EC:SEWALLI_renew
- P9: symbol USB_OTG -> USB_OTG-RESCUE-Meow_Meow
Changed lines of the file:
@@
 EESchema Schematic File Version 2
+LIBS:Meow Meow-rescue
 LIBS:power
 LIBS:device
@@
 F 0 "P7" H 10435 5070 60  0000 C CNN
 F 1 "KEY_UP_ARROW" H 10435 4870 60  0000 C CNN
-F 2 "Connectors:SEWALLI" H 10435 4970 60  0001 C CNN
+F 2 "Connectors_EC:SEWALLI_renew" H 10435 4970 60  0001 C CNN
 F 3 "" H 10435 4970 60  0001 C CNN
 	1    10435 4970
@@
 F 0 "P6" H 10125 5095 60  0000 C CNN
 F 1 "KEY_DOWN_ARROW" H 10125 4895 60  0000 C CNN
-F 2 "Connectors:SEWALLI" H 10125 4995 60  0001 C CNN
+F 2 "Connectors_EC:SEWALLI_renew" H 10125 4995 60  0001 C CNN
 F 3 "" H 10125 4995 60  0001 C CNN
 	1    10125 4995
@@
 F 0 "P3" H 9470 5100 60  0000 C CNN
 F 1 "KEY_RIGHT_ARROW" H 9470 4900 60  0000 C CNN
-F 2 "Connectors:SEWALLI" H 9470 5000 60  0001 C CNN
+F 2 "Connectors_EC:SEWALLI_renew" H 9470 5000 60  0001 C CNN
 F 3 "" H 9470 5000 60  0001 C CNN
 	1    9470 5000
@@
 F 0 "P2" H 9160 5100 60  0000 C CNN
 F 1 "SPACE" H 9160 4900 60  0000 C CNN
-F 2 "Connectors:SEWALLI" H 9160 5000 60  0001 C CNN
+F 2 "Connectors_EC:SEWALLI_renew" H 9160 5000 60  0001 C CNN
 F 3 "" H 9160 5000 60  0001 C CNN
 	1    9160 5000
@@
 F 0 "P5" H 9810 5100 60  0000 C CNN
 F 1 "KEY_LEFT_ARROW" H 9810 4900 60  0000 C CNN
-F 2 "Connectors:SEWALLI" H 9810 5000 60  0001 C CNN
+F 2 "Connectors_EC:SEWALLI_renew" H 9810 5000 60  0001 C CNN
 F 3 "" H 9810 5000 60  0001 C CNN
 	1    9810 5000
@@
 $EndComp
 $Comp
-L USB_OTG P9
+L USB_OTG-RESCUE-Meow_Meow P9
 U 1 1 5AFC70FD
 P 7935 3360
@@
 F 0 "P12" H 8660 5045 60  0000 C CNN
 F 1 "MOUSE_LEFT" H 8660 4845 60  0000 C CNN
-F 2 "Connectors:SEWALLI" H 8660 4945 60  0001 C CNN
+F 2 "Connectors_EC:SEWALLI_renew" H 8660 4945 60  0001 C CNN
 F 3 "" H 8660 4945 60  0001 C CNN
 	1    8660 4945
@@
 F 0 "P11" H 8380 5070 60  0000 C CNN
 F 1 "W" H 8380 4870 60  0000 C CNN
-F 2 "Connectors:SEWALLI" H 8380 4970 60  0001 C CNN
+F 2 "Connectors_EC:SEWALLI_renew" H 8380 4970 60  0001 C CNN
 F 3 "" H 8380 4970 60  0001 C CNN
 	1    8380 4970
@@
 F 0 "P8" H 7740 5070 60  0000 C CNN
 F 1 "S" H 7740 4870 60  0000 C CNN
-F 2 "Connectors:SEWALLI" H 7740 4970 60  0001 C CNN
+F 2 "Connectors_EC:SEWALLI_renew" H 7740 4970 60  0001 C CNN
 F 3 "" H 7740 4970 60  0001 C CNN
 	1    7740 4970
@@
 F 0 "P1" H 7355 5060 60  0000 C CNN
 F 1 "D" H 7355 4860 60  0000 C CNN
-F 2 "Connectors:SEWALLI" H 7355 4960 60  0001 C CNN
+F 2 "Connectors_EC:SEWALLI_renew" H 7355 4960 60  0001 C CNN
 F 3 "" H 7355 4960 60  0001 C CNN
 	1    7355 4960
@@
 F 0 "P10" H 8065 5075 60  0000 C CNN
 F 1 "A" H 8065 4875 60  0000 C CNN
-F 2 "Connectors:SEWALLI" H 8065 4975 60  0001 C CNN
+F 2 "Connectors_EC:SEWALLI_renew" H 8065 4975 60  0001 C CNN
 F 3 "" H 8065 4975 60  0001 C CNN
 	1    8065 4975

Commit message: Add logos
Parts:
- removed P13: Expansion, Pines:610X1221121, symbol CONN_02X06
- added P13, P14: CONN_01X06, Pines:61000618321, symbol CONN_01X06
- U1: value ATSAMD21G15A-AU -> ATSAMD21G18A-AU
Connections:
- net +3V3: now also P13.6 (P6)
- net CS: now also P14.2 (P2)
- net GND: now also P14.1 (P1)
- net I2S_D1/X7: now also P14.5 (P5)
- net I2S_SCK: now also P14.6 (P6)
- net MISO: now also P13.2 (P2)
- net MOSI: now also P13.1 (P1)
- net RX/X3: now also P14.3 (P3)
- net SCK: now also P13.3 (P3)
- net SCL: now also P13.5 (P5)
- net SDA: now also P13.4 (P4)
- net TX/X2: now also P14.4 (P4)
Changed lines of the file:
@@
 Title "Meow Meow"
 Date "2018-05-16"
-Rev "0.6"
+Rev "0.7"
 Comp "Electronic Cats"
 Comment1 "Andres Sabas"
@@
 P 3195 3255
 F 0 "U1" H 2595 4976 50  0000 L BNN
-F 1 "ATSAMD21G15A-AU" H 2594 1451 50  0000 L BNN
+F 1 "ATSAMD21G18A-AU" H 2594 1451 50  0000 L BNN
 F 2 "Housings_QFP:TQFP-48_7x7mm_Pitch0.5mm" H 3195 3255 50  0001 L BNN
 F 3 "3.01 USD" H 3195 3255 50  0001 L BNN
@@
 Text Notes 7805 5625 0    60   ~ 0
 PIN EXTRAS
-Text Label 9490 5760 0    60   ~ 0
+Text Label 9870 5730 0    60   ~ 0
 I2S_SCK
-Text Label 9495 5860 0    60   ~ 0
+Text Label 9875 5830 0    60   ~ 0
 I2S_D1/X7
-Text Label 9495 5960 0    60   ~ 0
+Text Label 9875 5930 0    60   ~ 0
 TX/X2
-Text Label 9495 6060 0    60   ~ 0
+Text Label 9875 6030 0    60   ~ 0
 RX/X3
 Text Label 8780 5760 2    60   ~ 0
@@
 Text Label 8780 5960 2    60   ~ 0
 SCK
-Text Label 9495 6160 0    60   ~ 0
+Text Label 9875 6130 0    60   ~ 0
 CS
 Text Label 8785 6060 2    60   ~ 0
@@
 L GND #PWR019
 U 1 1 5AFF5159
-P 9510 6260
-F 0 "#PWR019" H 9510 6010 50  0001 C CNN
-F 1 "GND" H 9510 6110 50  0000 C CNN
-F 2 "" H 9510 6260 50  0000 C CNN
-F 3 "" H 9510 6260 50  0000 C CNN
-	1    9510 6260
+P 9890 6230
+F 0 "#PWR019" H 9890 5980 50  0001 C CNN
+F 1 "GND" H 9890 6080 50  0000 C CNN
+F 2 "" H 9890 6230 50  0000 C CNN
+F 3 "" H 9890 6230 50  0000 C CNN
+	1    9890 6230
 	1    0    0    -1
 $EndComp
@@
 F 3 "" H 1590 1675 50  0000 C CNN
 	1    1590 1675
-	1    0    0    -1
-$EndComp
-$Comp
-L CONN_02X06 P13
-U 1 1 5B19929F
-P 9140 6010
-F 0 "P13" H 9140 6360 50  0000 C CNN
-F 1 "Expansion" H 9140 5660 50  0000 C CNN
-F 2 "Pines:610X1221121" H 9140 4810 50  0001 C CNN
-F 3 "" H 9140 4810 50  0000 C CNN
-	1    9140 6010
 	1    0    0    -1
 $EndComp
@@
 	8890 5760 8780 5760
 Wire Wire Line
-	9390 6160 9495 6160
-Wire Wire Line
-	9390 6060 9495 6060
-Wire Wire Line
-	9390 5960 9495 5960
-Wire Wire Line
-	9390 5860 9495 5860
-Wire Wire Line
-	9390 5760 9490 5760
+	9770 6130 9875 6130
+Wire Wire Line
+	9770 6030 9875 6030
+Wire Wire Line
+	9770 5930 9875 5930
+Wire Wire Line
+	9770 5830 9875 5830
+Wire Wire Line
+	9770 5730 9870 5730
 Wire Wire Line
 	8500 6260 8890 6260
 Wire Wire Line
-	9390 6260 9510 6260
+	9770 6230 9890 6230
 Wire Wire Line
 	9100 3285 8970 3285
@@
 Wire Wire Line
 	8745 3600 8745 3570
+$Comp
+L CONN_01X06 P13
+U 1 1 5B1DE3E8
+P 9090 6010
+F 0 "P13" H 9090 6360 50  0000 C CNN
+F 1 "CONN_01X06" V 9190 6010 50  0000 C CNN
+F 2 "Pines:61000618321" H 9090 6010 50  0001 C CNN
+F 3 "" H 9090 6010 50  0000 C CNN
+	1    9090 6010
+	1    0    0    -1
+$EndComp
+$Comp
+L CONN_01X06 P14
+U 1 1 5B1DE934
+P 9570 5980
+F 0 "P14" H 9570 6330 50  0000 C CNN
+F 1 "CONN_01X06" V 9670 5980 50  0000 C CNN
+F 2 "Pines:61000618321" H 9570 5980 50  0001 C CNN
+F 3 "" H 9570 5980 50  0000 C CNN
+	1    9570 5980
+	-1   0    0    1
+$EndComp
 $EndSCHEMATC

Commit message: Add pin 5v
Parts:
- removed P13, P14: CONN_01X06, Pines:61000618321, symbol CONN_01X06
- added P? (x2): CONN_01X07, symbol CONN_01X07
Connections:
- wire segments 97 -> 101
Changed lines of the file:
@@
 Title "Meow Meow"
 Date "2018-05-16"
-Rev "0.7"
+Rev "0.8"
 Comp "Electronic Cats"
 Comment1 "Andres Sabas"
@@
 	8745 3600 8745 3570
 $Comp
-L CONN_01X06 P13
-U 1 1 5B1DE3E8
-P 9090 6010
-F 0 "P13" H 9090 6360 50  0000 C CNN
-F 1 "CONN_01X06" V 9190 6010 50  0000 C CNN
-F 2 "Pines:61000618321" H 9090 6010 50  0001 C CNN
-F 3 "" H 9090 6010 50  0000 C CNN
-	1    9090 6010
-	1    0    0    -1
-$EndComp
-$Comp
-L CONN_01X06 P14
-U 1 1 5B1DE934
-P 9570 5980
-F 0 "P14" H 9570 6330 50  0000 C CNN
-F 1 "CONN_01X06" V 9670 5980 50  0000 C CNN
-F 2 "Pines:61000618321" H 9570 5980 50  0001 C CNN
-F 3 "" H 9570 5980 50  0000 C CNN
-	1    9570 5980
+L CONN_01X07 P?
+U 1 1 5B26BBAC
+P 9090 6060
+F 0 "P?" H 9090 6460 50  0000 C CNN
+F 1 "CONN_01X07" V 9190 6060 50  0000 C CNN
+F 2 "" H 9090 6060 50  0000 C CNN
+F 3 "" H 9090 6060 50  0000 C CNN
+	1    9090 6060
+	1    0    0    -1
+$EndComp
+$Comp
+L CONN_01X07 P?
+U 1 1 5B26BCF3
+P 9570 6030
+F 0 "P?" H 9570 6430 50  0000 C CNN
+F 1 "CONN_01X07" V 9670 6030 50  0000 C CNN
+F 2 "" H 9570 6030 50  0000 C CNN
+F 3 "" H 9570 6030 50  0000 C CNN
+	1    9570 6030
 	-1   0    0    1
 $EndComp
+Wire Wire Line
+	8355 6360 8890 6360
+$Comp
+L VCC #PWR?
+U 1 1 5B26C1A1
+P 8355 6340
+F 0 "#PWR?" H 8355 6190 50  0001 C CNN
+F 1 "VCC" H 8355 6490 50  0000 C CNN
+F 2 "" H 8355 6340 50  0000 C CNN
+F 3 "" H 8355 6340 50  0000 C CNN
+	1    8355 6340
+	1    0    0    -1
+$EndComp
+Wire Wire Line
+	8355 6360 8355 6340
+Wire Wire Line
+	9770 6330 9815 6330
+Wire Wire Line
+	9815 6330 9815 6230
+Connection ~ 9815 6230
 $EndSCHEMATC
