File: hardware/Meow Meow.sch (KiCad schematic (older format))
At the start: 28 parts, among them J1 SWD, J2 SWD, J3 SWD, P1 SPACE, P10 A, P11 W, P12 KEY_UP_ARROW, P2 KEY_DOWN_ARROW, P3 KEY_RIGHT_ARROW, P5 KEY_LEFT_ARROW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

Commit message: change connectors schematic
Parts:
- P9: footprint Connect:USB_Micro-B_10103594-0001LF -> Connector_USB:USB_Micro-B_Wuerth_629105150521
Connections:
- wire segments 104 -> 106
Changed lines of the file:
@@
 Text Label 8755 3395 2    60   ~ 0
 SWDIO
-Text Label 8760 3495 2    60   ~ 0
+Text Label 9470 3495 0    60   ~ 0
 SWCLK
 $Comp
 L MeowMeow:+3.3V #PWR06
 U 1 1 5AD9BCA9
-P 9470 3395
-F 0 "#PWR06" H 9470 3245 50  0001 C CNN
-F 1 "+3.3V" H 9470 3535 50  0000 C CNN
-F 2 "" H 9470 3395 50  0000 C CNN
-F 3 "" H 9470 3395 50  0000 C CNN
-	1    9470 3395
+P 8354 3477
+F 0 "#PWR06" H 8354 3327 50  0001 C CNN
+F 1 "+3.3V" H 8354 3617 50  0000 C CNN
+F 2 "" H 8354 3477 50  0000 C CNN
+F 3 "" H 8354 3477 50  0000 C CNN
+	1    8354 3477
 	1    0    0    -1
 $EndComp
@@
 L MeowMeow:GND #PWR07
 U 1 1 5AD9BD50
-P 9470 3495
-F 0 "#PWR07" H 9470 3245 50  0001 C CNN
-F 1 "GND" H 9475 3345 50  0000 C CNN
-F 2 "" H 9470 3495 50  0000 C CNN
-F 3 "" H 9470 3495 50  0000 C CNN
-	1    9470 3495
+P 9831 3431
+F 0 "#PWR07" H 9831 3181 50  0001 C CNN
+F 1 "GND" H 9836 3281 50  0000 C CNN
+F 2 "" H 9831 3431 50  0000 C CNN
+F 3 "" H 9831 3431 50  0000 C CNN
+	1    9831 3431
 	1    0    0    -1
 $EndComp
@@
 F 0 "P9" H 8260 3235 50  0000 C CNN
 F 1 "USB_Micro" H 7935 3560 50  0000 C CNN
-F 2 "Connect:USB_Micro-B_10103594-0001LF" V 7885 3260 50  0001 C CNN
+F 2 "Connector_USB:USB_Micro-B_Wuerth_629105150521" V 7885 3260 50  0001 C CNN
 F 3 "" V 7885 3260 50  0000 C CNN
 F 4 "629105150521" H 7935 3360 60  0001 C CNN "Part#"
@@
 NoConn ~ 2495 4655
 NoConn ~ 2495 4255
-Text Notes 7805 5625 0    60   ~ 0
+Text Notes 7745 5643 0    60   ~ 0
 PIN EXTRAS
 Text Label 10025 6130 0    60   ~ 0
 I2S_SCK
+Text Label 9340 6130 2    60   ~ 0
+I2S_D1/X7
 Text Label 10025 6030 0    60   ~ 0
-I2S_D1/X7
+TX/X2
+Text Label 9335 6030 2    60   ~ 0
+RX/X3
+Text Label 8346 5938 0    60   ~ 0
+MISO
+Text Label 7631 6038 2    60   ~ 0
+SCK
 Text Label 10020 5930 0    60   ~ 0
-TX/X2
-Text Label 9340 6130 2    60   ~ 0
-RX/X3
-Text Label 8105 6025 2    60   ~ 0
-MISO
-Text Label 8105 6125 2    60   ~ 0
-SCK
-Text Label 9335 6030 2    60   ~ 0
 CS
-Text Label 8820 5925 0    60   ~ 0
+Text Label 8341 6038 0    60   ~ 0
 SDA
-Text Label 8815 6025 0    60   ~ 0
+Text Label 7631 6138 2    60   ~ 0
 SCL
 $Comp
@@
 Wire Wire Line
 	8885 3395 8755 3395
-Wire Wire Line
-	8885 3495 8760 3495
 $Comp
 L MeowMeow:CONN_02X03 J2
@@
 	1    0    0    -1
 $EndComp
-Text Label 8105 5925 2    60   ~ 0
+Text Label 7631 5938 2    60   ~ 0
 MOSI
 $Comp
 L MeowMeow:CONN_02X03 J1
 U 1 1 5B57970D
-P 8440 6025
-F 0 "J1" H 8490 6225 50  0000 C CNN
-F 1 "SWD" H 8490 5825 50  0000 C CNN
-F 2 "Pin_Headers:Pin_Header_Straight_2x03_Pitch2.54mm_SMD" H 8440 6025 50  0001 C CNN
-F 3 "" H 8440 6025 50  0001 C CNN
-	1    8440 6025
-	1    0    0    -1
-$EndComp
-Wire Wire Line
-	8105 5925 8190 5925
-Wire Wire Line
-	8105 6025 8190 6025
-Wire Wire Line
-	8105 6125 8190 6125
+P 7966 6038
+F 0 "J1" H 8016 6238 50  0000 C CNN
+F 1 "SWD" H 8016 5838 50  0000 C CNN
+F 2 "Pin_Headers:Pin_Header_Straight_2x03_Pitch2.54mm_SMD" H 7966 6038 50  0001 C CNN
+F 3 "" H 7966 6038 50  0001 C CNN
+	1    7966 6038
+	1    0    0    -1
+$EndComp
+Wire Wire Line
+	7631 5938 7716 5938
+Wire Wire Line
+	7631 6038 7716 6038
+Wire Wire Line
+	7631 6138 7716 6138
 $Comp
 L MeowMeow:VCC #PWR021
 U 1 1 5B26C1A1
-P 8870 6125
-F 0 "#PWR021" H 8870 5975 50  0001 C CNN
-F 1 "VCC" H 8870 6265 50  0000 C CNN
-F 2 "" H 8870 6125 50  0000 C CNN
-F 3 "" H 8870 6125 50  0000 C CNN
-	1    8870 6125
-	-1   0    0    1
-$EndComp
-Wire Wire Line
-	8690 5925 8820 5925
-Wire Wire Line
-	8690 6025 8815 6025
-Wire Wire Line
-	8870 6125 8690 6125
+P 8623 6138
+F 0 "#PWR021" H 8623 5988 50  0001 C CNN
+F 1 "VCC" H 8623 6278 50  0000 C CNN
+F 2 "" H 8623 6138 50  0000 C CNN
+F 3 "" H 8623 6138 50  0000 C CNN
+	1    8623 6138
+	1    0    0    -1
+$EndComp
+Wire Wire Line
+	8216 5938 8346 5938
+Wire Wire Line
+	8216 6038 8341 6038
 Wire Wire Line
 	9940 5930 10020 5930
@@
 $EndComp
 Wire Wire Line
-	9385 3395 9470 3395
-Wire Wire Line
 	9385 3495 9470 3495
 Wire Wire Line
@@
 Wire Wire Line
 	9370 1290 9605 1290
+Wire Wire Line
+	8216 6138 8623 6138
+Wire Wire Line
+	8354 3495 8354 3477
+Wire Wire Line
+	8354 3495 8885 3495
+Wire Wire Line
+	9831 3395 9831 3431
+Wire Wire Line
+	9385 3395 9831 3395
 $EndSCHEMATC

Commit message: update files
Parts:
- C1, C2, C4, C5, C6: symbol MeowMeow:C_Small -> Meow-Meow-rescue:C_Small-MeowMeow
- D1, D2: symbol MeowMeow:LED -> Meow-Meow-rescue:LED-MeowMeow
- J1: value SWD -> Backpack1; symbol MeowMeow:CONN_02X03 -> Meow-Meow-rescue:CONN_02X03-MeowMeow
- J2: value SWD -> Backpack2; symbol MeowMeow:CONN_02X03 -> Meow-Meow-rescue:CONN_02X03-MeowMeow
- P1, P10, P11, P12, P2, P3, P5, P6, P7, P8: symbol MeowMeow:CONN_01X01_FEMALE -> Meow-Meow-rescue:CONN_01X01_FEMALE-MeowMeow
- P9: symbol MeowMeow:USB_OTG -> Meow-Meow-rescue:USB_OTG-MeowMeow
- R1, R2, R3: symbol MeowMeow:R_Small -> Meow-Meow-rescue:R_Small-MeowMeow
- SW1: symbol MeowMeow:SW_Push -> Meow-Meow-rescue:SW_Push-MeowMeow
- U1: symbol MeowMeow:ATSAMD21G18A-AU -> Meow-Meow-rescue:ATSAMD21G18A-AU-MeowMeow
- U2: symbol MeowMeow:AP2112 -> Meow-Meow-rescue:AP2112-MeowMeow
Changed lines of the file:
@@
 $EndDescr
 $Comp
-L MeowMeow:AP2112 U2
+L Meow-Meow-rescue:AP2112-MeowMeow U2
 U 1 1 5AD95D02
 P 8765 1490
@@
 NoConn ~ 7635 3460
 $Comp
-L MeowMeow:GND #PWR01
+L Meow-Meow-rescue:GND-MeowMeow #PWR01
 U 1 1 5AD96563
 P 7530 3600
@@
 $EndComp
 $Comp
-L MeowMeow:VCC #PWR02
+L Meow-Meow-rescue:VCC-MeowMeow #PWR02
 U 1 1 5AD96587
 P 7180 3135
@@
 SENSOR CAPACITIVE
 $Comp
-L MeowMeow:CONN_01X01_FEMALE P7
+L Meow-Meow-rescue:CONN_01X01_FEMALE-MeowMeow P7
 U 1 1 5AD981B5
 P 10435 4985
@@
 $EndComp
 $Comp
-L MeowMeow:CONN_01X01_FEMALE P6
+L Meow-Meow-rescue:CONN_01X01_FEMALE-MeowMeow P6
 U 1 1 5AD9829A
 P 10130 4985
@@
 $EndComp
 $Comp
-L MeowMeow:CONN_01X01_FEMALE P3
+L Meow-Meow-rescue:CONN_01X01_FEMALE-MeowMeow P3
 U 1 1 5AD98302
 P 9485 4995
@@
 $EndComp
 $Comp
-L MeowMeow:CONN_01X01_FEMALE P2
+L Meow-Meow-rescue:CONN_01X01_FEMALE-MeowMeow P2
 U 1 1 5AD9836F
 P 9155 5005
@@
 Y4
 $Comp
-L MeowMeow:C_Small C4
+L Meow-Meow-rescue:C_Small-MeowMeow C4
 U 1 1 5AD98E8E
 P 8030 1440
@@
 $EndComp
 $Comp
-L MeowMeow:C_Small C5
+L Meow-Meow-rescue:C_Small-MeowMeow C5
 U 1 1 5AD98EFB
 P 9370 1455
@@
 $EndComp
 $Comp
-L MeowMeow:C_Small C6
+L Meow-Meow-rescue:C_Small-MeowMeow C6
 U 1 1 5AD98F7F
 P 9605 1455
@@
 $EndComp
 $Comp
-L MeowMeow:LED D1
+L Meow-Meow-rescue:LED-MeowMeow D1
 U 1 1 5AD9907D
 P 10560 3100
@@
 $EndComp
 $Comp
-L MeowMeow:R_Small R2
+L Meow-Meow-rescue:R_Small-MeowMeow R2
 U 1 1 5AD9913C
 P 10230 3100
@@
 $EndComp
 $Comp
-L MeowMeow:GND #PWR03
+L Meow-Meow-rescue:GND-MeowMeow #PWR03
 U 1 1 5AD99661
 P 10055 3100
@@
 $EndComp
 $Comp
-L MeowMeow:+3.3V #PWR04
+L Meow-Meow-rescue:+3.3V-MeowMeow #PWR04
 U 1 1 5AD9971F
 P 10790 3100
@@
 $EndComp
 $Comp
-L MeowMeow:LED D2
+L Meow-Meow-rescue:LED-MeowMeow D2
 U 1 1 5AD99995
 P 10560 3515
@@
 $EndComp
 $Comp
-L MeowMeow:R_Small R3
+L Meow-Meow-rescue:R_Small-MeowMeow R3
 U 1 1 5AD9999C
 P 10230 3515
@@
 $EndComp
 $Comp
-L MeowMeow:GND #PWR05
+L Meow-Meow-rescue:GND-MeowMeow #PWR05
 U 1 1 5AD999A6
 P 10055 3515
@@
 SWCLK
 $Comp
-L MeowMeow:+3.3V #PWR06
+L Meow-Meow-rescue:+3.3V-MeowMeow #PWR06
 U 1 1 5AD9BCA9
 P 8354 3477
@@
 $EndComp
 $Comp
-L MeowMeow:GND #PWR07
+L Meow-Meow-rescue:GND-MeowMeow #PWR07
 U 1 1 5AD9BD50
 P 9831 3431
@@
 $EndComp
 $Comp
-L MeowMeow:R_Small R1
+L Meow-Meow-rescue:R_Small-MeowMeow R1
 U 1 1 5AD9C752
 P 2215 1655
@@
 $EndComp
 $Comp
-L MeowMeow:CONN_01X01_FEMALE P5
+L Meow-Meow-rescue:CONN_01X01_FEMALE-MeowMeow P5
 U 1 1 5AD9D9AC
 P 9795 4995
@@
 Y2
 $Comp
-L MeowMeow:GND #PWR08
+L Meow-Meow-rescue:GND-MeowMeow #PWR08
 U 1 1 5ADA067C
 P 8030 1600
@@
 $EndComp
 $Comp
-L MeowMeow:GND #PWR09
+L Meow-Meow-rescue:GND-MeowMeow #PWR09
 U 1 1 5ADA0DDC
 P 8250 1720
@@
 $EndComp
 $Comp
-L MeowMeow:VCC #PWR010
+L Meow-Meow-rescue:VCC-MeowMeow #PWR010
 U 1 1 5ADA0F24
 P 7590 1175
@@
 $EndComp
 $Comp
-L MeowMeow:+3.3V #PWR011
+L Meow-Meow-rescue:+3.3V-MeowMeow #PWR011
 U 1 1 5ADA11F4
 P 9945 1225
@@
 $EndComp
 $Comp
-L MeowMeow:GND #PWR012
+L Meow-Meow-rescue:GND-MeowMeow #PWR012
 U 1 1 5ADA139A
 P 9605 1630
@@
 $EndComp
 $Comp
-L MeowMeow:GND #PWR013
+L Meow-Meow-rescue:GND-MeowMeow #PWR013
 U 1 1 5ADA141E
 P 9370 1630
@@
 $EndComp
 $Comp
-L MeowMeow:GND #PWR014
+L Meow-Meow-rescue:GND-MeowMeow #PWR014
 U 1 1 5AE3E770
 P 8035 3760
@@
 SCL
 $Comp
-L MeowMeow:ATSAMD21G18A-AU U1
+L Meow-Meow-rescue:ATSAMD21G18A-AU-MeowMeow U1
 U 1 1 5AFC6E86
 P 3195 3255
@@
 $EndComp
 $Comp
-L MeowMeow:USB_OTG P9
+L Meow-Meow-rescue:USB_OTG-MeowMeow P9
 U 1 1 5AFC70FD
 P 7935 3360
@@
 Y9
 $Comp
-L MeowMeow:C_Small C1
+L Meow-Meow-rescue:C_Small-MeowMeow C1
 U 1 1 5AFCC5C3
 P 3945 2185
@@
 $EndComp
 $Comp
-L MeowMeow:GND #PWR015
+L Meow-Meow-rescue:GND-MeowMeow #PWR015
 U 1 1 5AFCC90C
 P 3945 2340
@@
 $EndComp
 $Comp
-L MeowMeow:+3.3V #PWR016
+L Meow-Meow-rescue:+3.3V-MeowMeow #PWR016
 U 1 1 5AFCCDC2
 P 3990 1565
@@
 $EndComp
 $Comp
-L MeowMeow:C_Small C2
+L Meow-Meow-rescue:C_Small-MeowMeow C2
 U 1 1 5AFCCE9C
 P 4210 1755
@@
 $EndComp
 $Comp
-L MeowMeow:GND #PWR017
+L Meow-Meow-rescue:GND-MeowMeow #PWR017
 U 1 1 5AFCCF73
 P 4210 1885
@@
 $EndComp
 $Comp
-L MeowMeow:GND #PWR018
+L Meow-Meow-rescue:GND-MeowMeow #PWR018
 U 1 1 5AFCF78D
 P 4025 4740
@@
 $EndComp
 $Comp
-L MeowMeow:CONN_01X01_FEMALE P12
+L Meow-Meow-rescue:CONN_01X01_FEMALE-MeowMeow P12
 U 1 1 5AFCFBC0
 P 8840 5005
@@
 $EndComp
 $Comp
-L MeowMeow:CONN_01X01_FEMALE P11
+L Meow-Meow-rescue:CONN_01X01_FEMALE-MeowMeow P11
 U 1 1 5AFCFBC7
 P 8570 5005
@@
 $EndComp
 $Comp
-L MeowMeow:CONN_01X01_FEMALE P8
+L Meow-Meow-rescue:CONN_01X01_FEMALE-MeowMeow P8
 U 1 1 5AFCFBCE
 P 7990 5015
@@
 $EndComp
 $Comp
-L MeowMeow:CONN_01X01_FEMALE P1
+L Meow-Meow-rescue:CONN_01X01_FEMALE-MeowMeow P1
 U 1 1 5AFCFBD5
 P 7685 5005
@@
 Y15
 $Comp
-L MeowMeow:CONN_01X01_FEMALE P10
+L Meow-Meow-rescue:CONN_01X01_FEMALE-MeowMeow P10
 U 1 1 5AFCFBE0
 P 8290 5010
@@
 SCL
 $Comp
-L MeowMeow:GND #PWR019
+L Meow-Meow-rescue:GND-MeowMeow #PWR019
 U 1 1 5AFF5159
 P 9335 5930
@@
 $EndComp
 $Comp
-L MeowMeow:SW_Push SW1
+L Meow-Meow-rescue:SW_Push-MeowMeow SW1
 U 1 1 5B071A82
 P 1835 1655
@@
 $EndComp
 $Comp
-L MeowMeow:GND #PWR020
+L Meow-Meow-rescue:GND-MeowMeow #PWR020
 U 1 1 5B0727F0
 P 1590 1675
@@
 	8885 3395 8755 3395
 $Comp
-L MeowMeow:CONN_02X03 J2
+L Meow-Meow-rescue:CONN_02X03-MeowMeow J2
 U 1 1 5B57974D
 P 9690 6030
 F 0 "J2" H 9740 6230 50  0000 C CNN
-F 1 "SWD" H 9740 5830 50  0000 C CNN
+F 1 "Backpack2" H 9740 5830 50  0000 C CNN
 F 2 "Pin_Headers:Pin_Header_Straight_2x03_Pitch2.54mm_SMD" H 9690 6030 50  0001 C CNN
 F 3 "" H 9690 6030 50  0001 C CNN
@@
 MOSI
 $Comp
-L MeowMeow:CONN_02X03 J1
+L Meow-Meow-rescue:CONN_02X03-MeowMeow J1
 U 1 1 5B57970D
 P 7966 6038
 F 0 "J1" H 8016 6238 50  0000 C CNN
-F 1 "SWD" H 8016 5838 50  0000 C CNN
+F 1 "Backpack1" H 8016 5838 50  0000 C CNN
 F 2 "Pin_Headers:Pin_Header_Straight_2x03_Pitch2.54mm_SMD" H 7966 6038 50  0001 C CNN
 F 3 "" H 7966 6038 50  0001 C CNN
@@
 	7631 6138 7716 6138
 $Comp
-L MeowMeow:VCC #PWR021
+L Meow-Meow-rescue:VCC-MeowMeow #PWR021
 U 1 1 5B26C1A1
 P 8623 6138

Commit message: change reset button
Parts:
- SW1: footprint Buttons_Switches_SMD:SW_SPST_B3U-1000P-B -> Buttons_Switches_SMD:SW_SPST_TL3342
Changed lines of the file:
@@
 Sheet 1 1
 Title "Meow Meow"
-Date "2018-08-19"
-Rev "1.1"
+Date "2019-04-01"
+Rev "1.2"
 Comp "Electronic Cats"
 Comment1 "Andres Sabas"
@@
 F 0 "SW1" H 1885 1755 50  0000 L CNN
 F 1 "SW_Push" H 1835 1595 50  0000 C CNN
-F 2 "Buttons_Switches_SMD:SW_SPST_B3U-1000P-B" H 1835 1855 50  0001 C CNN
+F 2 "Buttons_Switches_SMD:SW_SPST_TL3342" H 1835 1855 50  0001 C CNN
 F 3 "" H 1835 1855 50  0000 C CNN
 	1    1835 1655

Commit message: Update 1.3
Parts:
- removed R1: 330, Resistors_SMD:R_0805_HandSoldering, symbol Meow-Meow-rescue:R_Small-MeowMeow
- P9: footprint Connector_USB:USB_Micro-B_Wuerth_629105150521 -> Connectors:U254051N4BH806; Part# 629105150521 -> U254-051N-4BH806
- U1: Part# ATSAMD21G15A-AU -> ATSAMD21G18A-AU
Connections:
- wire segments 106 -> 105
Changed lines of the file:
@@
 EESchema Schematic File Version 4
 LIBS:Meow Meow-cache
-EELAYER 26 0
+EELAYER 29 0
 EELAYER END
 $Descr A4 11693 8268
@@
 Sheet 1 1
 Title "Meow Meow"
-Date "2019-04-01"
-Rev "1.2"
+Date "2019-11-14"
+Rev "1.3"
 Comp "Electronic Cats"
 Comment1 "Andres Sabas"
@@
 $EndComp
 $Comp
-L Meow-Meow-rescue:R_Small-MeowMeow R1
-U 1 1 5AD9C752
-P 2215 1655
-F 0 "R1" V 2280 1580 50  0000 L CNN
-F 1 "330" V 2150 1585 50  0000 L CNN
-F 2 "Resistors_SMD:R_0805_HandSoldering" H 2215 1655 50  0001 C CNN
-F 3 "" H 2215 1655 50  0000 C CNN
-F 4 "B3U-1000P" V 2215 1655 60  0001 C CNN "Part#"
-	1    2215 1655
-	0    -1   -1   0
-$EndComp
-$Comp
 L Meow-Meow-rescue:CONN_01X01_FEMALE-MeowMeow P5
 U 1 1 5AD9D9AC
@@
 F 5 "TQFP-48 Microchip" H 3195 3255 50  0001 L BNN "Campo5"
 F 6 "SAMD21G Series 256 kB Flash 32 kB SRAM 48 MHz 32-Bit Microcontroller - TQFP-48" H 3195 3255 50  0001 L BNN "Campo6"
-F 7 "ATSAMD21G15A-AU" H 3195 3255 50  0001 L BNN "Part#"
+F 7 "ATSAMD21G18A-AU" H 3195 3255 50  0001 L BNN "Part#"
 	1    3195 3255
 	1    0    0    -1
@@
 F 0 "P9" H 8260 3235 50  0000 C CNN
 F 1 "USB_Micro" H 7935 3560 50  0000 C CNN
-F 2 "Connector_USB:USB_Micro-B_Wuerth_629105150521" V 7885 3260 50  0001 C CNN
+F 2 "Connectors:U254051N4BH806" V 7885 3260 50  0001 C CNN
 F 3 "" V 7885 3260 50  0000 C CNN
-F 4 "629105150521" H 7935 3360 60  0001 C CNN "Part#"
+F 4 "U254-051N-4BH806" H 7935 3360 60  0001 C CNN "Part#"
 	1    7935 3360
 	0    1    1    0
@@
 $EndComp
 $Comp
-L Meow-Meow-rescue:SW_Push-MeowMeow SW1
-U 1 1 5B071A82
-P 1835 1655
-F 0 "SW1" H 1885 1755 50  0000 L CNN
-F 1 "SW_Push" H 1835 1595 50  0000 C CNN
-F 2 "Buttons_Switches_SMD:SW_SPST_TL3342" H 1835 1855 50  0001 C CNN
-F 3 "" H 1835 1855 50  0000 C CNN
-	1    1835 1655
-	1    0    0    -1
-$EndComp
-$Comp
 L Meow-Meow-rescue:GND-MeowMeow #PWR020
 U 1 1 5B0727F0
@@
 Wire Wire Line
 	3895 4355 4025 4355
-Wire Wire Line
-	2495 1655 2315 1655
 Wire Wire Line
 	2495 4855 2295 4855
@@
 	11215 5515 11215 5520
 Wire Wire Line
-	2115 1655 2035 1655
-Wire Wire Line
 	1635 1655 1590 1655
 Wire Wire Line
@@
 Wire Wire Line
 	9385 3395 9831 3395
+$Comp
+L Meow-Meow-rescue:SW_Push-MeowMeow SW1
+U 1 1 5B071A82
+P 1835 1655
+F 0 "SW1" H 1885 1755 50  0000 L CNN
+F 1 "SW_Push" H 1835 1595 50  0000 C CNN
+F 2 "Buttons_Switches_SMD:SW_SPST_TL3342" H 1835 1855 50  0001 C CNN
+F 3 "" H 1835 1855 50  0000 C CNN
+	1    1835 1655
+	1    0    0    -1
+$EndComp
+Wire Wire Line
+	2035 1655 2495 1655
 $EndSCHEMATC

Commit message: update schematic headers feather
Parts:
- removed J1: Backpack1, Pin_Headers:Pin_Header_Straight_2x03_Pitch2.54mm_SMD, symbol Meow-Meow-rescue:CONN_02X03-MeowMeow
- removed J2: Backpack2, Pin_Headers:Pin_Header_Straight_2x03_Pitch2.54mm_SMD, symbol Meow-Meow-rescue:CONN_02X03-MeowMeow
- removed U2: AP2114-3.3K, TO_SOT_Packages_SMD:SOT-223-3_TabPin2, symbol Meow-Meow-rescue:AP2112-MeowMeow
- added J1: Conn_Left, Connector_PinSocket_2.54mm:PinSocket_1x16_P2.54mm_Vertical_SMD_Pin1Left, symbol Connector_Generic:Conn_01x16
- added J2: Conn_Right, Connector_PinSocket_2.54mm:PinSocket_1x12_P2.54mm_Vertical_SMD_Pin1Right, symbol Connector_Generic:Conn_01x12
- added R1: 10K, Resistor_SMD:R_0805_2012Metric_Pad1.15x1.40mm_HandSolder, symbol Device:R_Small
- added U2: AP2112K-3.3, Package_TO_SOT_SMD:SOT-23-5, symbol Regulator_Linear:AP2112K-3.3
- SW1: value SW_Push -> RESET
Connections:
- net labels added: +BATT, EN, GPIO05, GPIO06, GPIO08, GPIO09, GPIO10, GPIO11, GPIO12, GPIO13, MISC, RESET, RX_X3, TX_X2, VBUS
- net labels removed: CS, D8, I2S_D1/X7, I2S_SCK, RX/X3, TX/X2, VCC
- wire segments 105 -> 133
- no-connect marks 14 -> 10
Other:
- note added: "Analog A0-A5"
- note added: "Aref"

Commit message: update pinout and simbol
Parts:
- removed J3: SWD, Pin_Headers:Pin_Header_Straight_2x02_Pitch2.54mm_SMD, symbol Connector_Generic:Conn_02x02_Counter_Clockwise
- removed U1: ATSAMD21G18A-AU, Housings_QFP:TQFP-48_7x7mm_Pitch0.5mm, symbol Meow-Meow-rescue:ATSAMD21G18A-AU-MeowMeow
- added J3: SWD, symbol Connector_Generic:Conn_01x04
- added U1: ATSAMD21G18A-M, Package_DFN_QFN:QFN-48-1EP_7x7mm_P0.5mm_EP5.15x5.15mm, symbol MCU_Microchip_SAMD:ATSAMD21G18A-M
- C1, C2, C4, C5, C6: symbol Meow-Meow-rescue:C_Small-MeowMeow -> Meow-Meow-rescue:C_Small-MeowMeow-Meow-Meow-rescue
- D1, D2: symbol Meow-Meow-rescue:LED-MeowMeow -> Meow-Meow-rescue:LED-MeowMeow-Meow-Meow-rescue
- P1, P10, P11, P12, P2, P3, P5, P6, P7, P8: symbol Meow-Meow-rescue:CONN_01X01_FEMALE-MeowMeow -> Meow-Meow-rescue:CONN_01X01_FEMALE-MeowMeow-Meow-Meow-rescue
- P9: symbol Meow-Meow-rescue:USB_OTG-MeowMeow -> Meow-Meow-rescue:USB_OTG-MeowMeow-Meow-Meow-rescue
- R2, R3: symbol Meow-Meow-rescue:R_Small-MeowMeow -> Meow-Meow-rescue:R_Small-MeowMeow-Meow-Meow-rescue
- SW1: symbol Meow-Meow-rescue:SW_Push-MeowMeow -> Meow-Meow-rescue:SW_Push-MeowMeow-Meow-Meow-rescue
- U2: symbol Regulator_Linear:AP2112K-3.3 -> Meow-Meow-rescue:AP2112K-3.3-Regulator_Linear-Meow-Meow-rescue
Connections:
- net labels added: A0, A1, A2, A3, CS, RX, TX
- net labels removed: RX_X3, TX_X2
- wire segments 133 -> 134
- no-connect marks 10 -> 8
Other:
- note added: "Analog A0-A3"
- note removed: "Analog A0-A5"
- note removed: "Aref"
