File: hardware/Meow Meow.sch (KiCad schematic (older format))
At the start: 28 parts, among them J1 Conn_Left, J2 Conn_Right, J3 SWD, P1 SPACE, P10 A, P11 W, P12 KEY_UP_ARROW, P2 KEY_DOWN_ARROW, P3 KEY_RIGHT_ARROW, P5 KEY_LEFT_ARROW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

Commit message: change GPIO13
Parts:
- C1, C2, C4, C5, C6: symbol Meow-Meow-rescue:C_Small-MeowMeow-Meow-Meow-rescue -> Meow-Meow-rescue:C_Small-MeowMeow-Meow-Meow-rescue-Meow-Meow-rescue
- D1, D2: symbol Meow-Meow-rescue:LED-MeowMeow-Meow-Meow-rescue -> Meow-Meow-rescue:LED-MeowMeow-Meow-Meow-rescue-Meow-Meow-rescue
- P1, P10, P11, P12, P2, P3, P5, P6, P7, P8: symbol Meow-Meow-rescue:CONN_01X01_FEMALE-MeowMeow-Meow-Meow-rescue -> Meow-Meow-rescue:CONN_01X01_FEMALE-MeowMeow-Meow-Meow-rescue-Meow-Meow-rescue
- P9: symbol Meow-Meow-rescue:USB_OTG-MeowMeow-Meow-Meow-rescue -> Meow-Meow-rescue:USB_OTG-MeowMeow-Meow-Meow-rescue-Meow-Meow-rescue
- R2, R3: symbol Meow-Meow-rescue:R_Small-MeowMeow-Meow-Meow-rescue -> Meow-Meow-rescue:R_Small-MeowMeow-Meow-Meow-rescue-Meow-Meow-rescue
- SW1: symbol Meow-Meow-rescue:SW_Push-MeowMeow-Meow-Meow-rescue -> Meow-Meow-rescue:SW_Push-MeowMeow-Meow-Meow-rescue-Meow-Meow-rescue
- U2: symbol Meow-Meow-rescue:AP2112K-3.3-Regulator_Linear-Meow-Meow-rescue -> Meow-Meow-rescue:AP2112K-3.3-Regulator_Linear-Meow-Meow-rescue-Meow-Meow-rescue
Connections:
- net labels removed: +BATT, CS
- wire segments 134 -> 133
- no-connect marks 8 -> 10
Changed lines of the file:
@@
 NoConn ~ 7635 3460
 $Comp
-L Meow-Meow-rescue:GND-MeowMeow-Meow-Meow-rescue #PWR01
+L Meow-Meow-rescue:GND-MeowMeow-Meow-Meow-rescue-Meow-Meow-rescue #PWR01
 U 1 1 5AD96563
 P 7530 3600
@@
 SENSOR CAPACITIVE
 $Comp
-L Meow-Meow-rescue:CONN_01X01_FEMALE-MeowMeow-Meow-Meow-rescue P7
+L Meow-Meow-rescue:CONN_01X01_FEMALE-MeowMeow-Meow-Meow-rescue-Meow-Meow-rescue P7
 U 1 1 5AD981B5
 P 10455 5616
@@
 $EndComp
 $Comp
-L Meow-Meow-rescue:CONN_01X01_FEMALE-MeowMeow-Meow-Meow-rescue P6
+L Meow-Meow-rescue:CONN_01X01_FEMALE-MeowMeow-Meow-Meow-rescue-Meow-Meow-rescue P6
 U 1 1 5AD9829A
 P 10150 5616
@@
 $EndComp
 $Comp
-L Meow-Meow-rescue:CONN_01X01_FEMALE-MeowMeow-Meow-Meow-rescue P3
+L Meow-Meow-rescue:CONN_01X01_FEMALE-MeowMeow-Meow-Meow-rescue-Meow-Meow-rescue P3
 U 1 1 5AD98302
 P 9505 5626
@@
 $EndComp
 $Comp
-L Meow-Meow-rescue:CONN_01X01_FEMALE-MeowMeow-Meow-Meow-rescue P2
+L Meow-Meow-rescue:CONN_01X01_FEMALE-MeowMeow-Meow-Meow-rescue-Meow-Meow-rescue P2
 U 1 1 5AD9836F
 P 9175 5636
@@
 Y4
 $Comp
-L Meow-Meow-rescue:C_Small-MeowMeow-Meow-Meow-rescue C4
+L Meow-Meow-rescue:C_Small-MeowMeow-Meow-Meow-rescue-Meow-Meow-rescue C4
 U 1 1 5AD98E8E
 P 8030 1440
@@
 $EndComp
 $Comp
-L Meow-Meow-rescue:LED-MeowMeow-Meow-Meow-rescue D1
+L Meow-Meow-rescue:LED-MeowMeow-Meow-Meow-rescue-Meow-Meow-rescue D1
 U 1 1 5AD9907D
 P 10560 3100
@@
 $EndComp
 $Comp
-L Meow-Meow-rescue:R_Small-MeowMeow-Meow-Meow-rescue R2
+L Meow-Meow-rescue:R_Small-MeowMeow-Meow-Meow-rescue-Meow-Meow-rescue R2
 U 1 1 5AD9913C
 P 10230 3100
@@
 $EndComp
 $Comp
-L Meow-Meow-rescue:GND-MeowMeow-Meow-Meow-rescue #PWR03
+L Meow-Meow-rescue:GND-MeowMeow-Meow-Meow-rescue-Meow-Meow-rescue #PWR03
 U 1 1 5AD99661
 P 10055 3100
@@
 $EndComp
 $Comp
-L Meow-Meow-rescue:+3.3V-MeowMeow-Meow-Meow-rescue #PWR04
+L Meow-Meow-rescue:+3.3V-MeowMeow-Meow-Meow-rescue-Meow-Meow-rescue #PWR04
 U 1 1 5AD9971F
 P 10790 3100
@@
 $EndComp
 $Comp
-L Meow-Meow-rescue:LED-MeowMeow-Meow-Meow-rescue D2
+L Meow-Meow-rescue:LED-MeowMeow-Meow-Meow-rescue-Meow-Meow-rescue D2
 U 1 1 5AD99995
 P 10560 3515
@@
 $EndComp
 $Comp
-L Meow-Meow-rescue:R_Small-MeowMeow-Meow-Meow-rescue R3
+L Meow-Meow-rescue:R_Small-MeowMeow-Meow-Meow-rescue-Meow-Meow-rescue R3
 U 1 1 5AD9999C
 P 10230 3515
@@
 $EndComp
 $Comp
-L Meow-Meow-rescue:GND-MeowMeow-Meow-Meow-rescue #PWR05
+L Meow-Meow-rescue:GND-MeowMeow-Meow-Meow-rescue-Meow-Meow-rescue #PWR05
 U 1 1 5AD999A6
 P 10055 3515
@@
 SWCLK
 $Comp
-L Meow-Meow-rescue:+3.3V-MeowMeow-Meow-Meow-rescue #PWR06
+L Meow-Meow-rescue:+3.3V-MeowMeow-Meow-Meow-rescue-Meow-Meow-rescue #PWR06
 U 1 1 5AD9BCA9
 P 8865 3280
@@
 $EndComp
 $Comp
-L Meow-Meow-rescue:GND-MeowMeow-Meow-Meow-rescue #PWR07
+L Meow-Meow-rescue:GND-MeowMeow-Meow-Meow-rescue-Meow-Meow-rescue #PWR07
 U 1 1 5AD9BD50
 P 8870 3580
@@
 $EndComp
 $Comp
-L Meow-Meow-rescue:CONN_01X01_FEMALE-MeowMeow-Meow-Meow-rescue P5
+L Meow-Meow-rescue:CONN_01X01_FEMALE-MeowMeow-Meow-Meow-rescue-Meow-Meow-rescue P5
 U 1 1 5AD9D9AC
 P 9815 5626
@@
 Y2
 $Comp
-L Meow-Meow-rescue:GND-MeowMeow-Meow-Meow-rescue #PWR08
+L Meow-Meow-rescue:GND-MeowMeow-Meow-Meow-rescue-Meow-Meow-rescue #PWR08
 U 1 1 5ADA067C
 P 8030 1600
@@
 $EndComp
 $Comp
-L Meow-Meow-rescue:GND-MeowMeow-Meow-Meow-rescue #PWR09
+L Meow-Meow-rescue:GND-MeowMeow-Meow-Meow-rescue-Meow-Meow-rescue #PWR09
 U 1 1 5ADA0DDC
 P 8615 1725
@@
 $EndComp
 $Comp
-L Meow-Meow-rescue:GND-MeowMeow-Meow-Meow-rescue #PWR014
+L Meow-Meow-rescue:GND-MeowMeow-Meow-Meow-rescue-Meow-Meow-rescue #PWR014
 U 1 1 5AE3E770
 P 8035 3760
@@
 SCL
 $Comp
-L Meow-Meow-rescue:USB_OTG-MeowMeow-Meow-Meow-rescue P9
+L Meow-Meow-rescue:USB_OTG-MeowMeow-Meow-Meow-rescue-Meow-Meow-rescue P9
 U 1 1 5AFC70FD
 P 7935 3360
@@
 Y9
 $Comp
-L Meow-Meow-rescue:+3.3V-MeowMeow-Meow-Meow-rescue #PWR016
+L Meow-Meow-rescue:+3.3V-MeowMeow-Meow-Meow-rescue-Meow-Meow-rescue #PWR016
 U 1 1 5AFCCDC2
 P 2740 1060
@@
 $EndComp
 $Comp
-L Meow-Meow-rescue:C_Small-MeowMeow-Meow-Meow-rescue C2
+L Meow-Meow-rescue:C_Small-MeowMeow-Meow-Meow-rescue-Meow-Meow-rescue C2
 U 1 1 5AFCCE9C
 P 3140 845
@@
 $EndComp
 $Comp
-L Meow-Meow-rescue:GND-MeowMeow-Meow-Meow-rescue #PWR017
+L Meow-Meow-rescue:GND-MeowMeow-Meow-Meow-rescue-Meow-Meow-rescue #PWR017
 U 1 1 5AFCCF73
 P 3270 845
@@
 $EndComp
 $Comp
-L Meow-Meow-rescue:GND-MeowMeow-Meow-Meow-rescue #PWR018
+L Meow-Meow-rescue:GND-MeowMeow-Meow-Meow-rescue-Meow-Meow-rescue #PWR018
 U 1 1 5AFCF78D
 P 2790 4990
@@
 $EndComp
 $Comp
-L Meow-Meow-rescue:CONN_01X01_FEMALE-MeowMeow-Meow-Meow-rescue P12
+L Meow-Meow-rescue:CONN_01X01_FEMALE-MeowMeow-Meow-Meow-rescue-Meow-Meow-rescue P12
 U 1 1 5AFCFBC0
 P 8860 5636
@@
 $EndComp
 $Comp
-L Meow-Meow-rescue:CONN_01X01_FEMALE-MeowMeow-Meow-Meow-rescue P11
+L Meow-Meow-rescue:CONN_01X01_FEMALE-MeowMeow-Meow-Meow-rescue-Meow-Meow-rescue P11
 U 1 1 5AFCFBC7
 P 8590 5636
@@
 $EndComp
 $Comp
-L Meow-Meow-rescue:CONN_01X01_FEMALE-MeowMeow-Meow-Meow-rescue P8
+L Meow-Meow-rescue:CONN_01X01_FEMALE-MeowMeow-Meow-Meow-rescue-Meow-Meow-rescue P8
 U 1 1 5AFCFBCE
 P 8010 5646
@@
 $EndComp
 $Comp
-L Meow-Meow-rescue:CONN_01X01_FEMALE-MeowMeow-Meow-Meow-rescue P1
+L Meow-Meow-rescue:CONN_01X01_FEMALE-MeowMeow-Meow-Meow-rescue-Meow-Meow-rescue P1
 U 1 1 5AFCFBD5
 P 7705 5636
@@
 Y15
 $Comp
-L Meow-Meow-rescue:CONN_01X01_FEMALE-MeowMeow-Meow-Meow-rescue P10
+L Meow-Meow-rescue:CONN_01X01_FEMALE-MeowMeow-Meow-Meow-rescue-Meow-Meow-rescue P10
 U 1 1 5AFCFBE0
 P 8310 5641
@@
 Text Label 1930 3115 2    50   ~ 0
 GPIO10
-Text Label 3530 2515 0    50   ~ 0
+Text Label 1915 3715 2    50   ~ 0
 GPIO13
 Text Label 1930 3215 2    50   ~ 0
@@
 PIN EXTRAS
 $Comp
-L Meow-Meow-rescue:GND-MeowMeow-Meow-Meow-rescue #PWR020
+L Meow-Meow-rescue:GND-MeowMeow-Meow-Meow-rescue-Meow-Meow-rescue #PWR020
 U 1 1 5B0727F0
 P 4775 1690
@@
 	3040 1065 3040 845
 $Comp
-L Meow-Meow-rescue:SW_Push-MeowMeow-Meow-Meow-rescue SW1
+L Meow-Meow-rescue:SW_Push-MeowMeow-Meow-Meow-rescue-Meow-Meow-rescue SW1
 U 1 1 5B071A82
 P 5020 1670
@@
 MISC
 $Comp
-L power:+BATT #PWR0103
-U 1 1 5D53E0CA
-P 4225 5945
-F 0 "#PWR0103" H 4225 5795 50  0001 C CNN
-F 1 "+BATT" H 4225 6095 50  0000 C CNN
-F 2 "" H 4225 5945 50  0001 C CNN
-F 3 "" H 4225 5945 50  0001 C CNN
-	1    4225 5945
-	1    0    0    -1
-$EndComp
-$Comp
 L power:VBUS #PWR0104
 U 1 1 5D53E609
@@
 Wire Wire Line
 	3075 5895 3075 6095
-Wire Wire Line
-	4225 5995 4225 5945
 Wire Wire Line
 	4475 5945 4475 6195
@@
 Analog A0-A3
 $Comp
-L Meow-Meow-rescue:AP2112K-3.3-Regulator_Linear-Meow-Meow-rescue U2
+L Meow-Meow-rescue:AP2112K-3.3-Regulator_Linear-Meow-Meow-rescue-Meow-Meow-rescue U2
 U 1 1 5E539C42
 P 8615 1390
@@
 	9255 1555 9255 1630
 $Comp
-L Meow-Meow-rescue:GND-MeowMeow-Meow-Meow-rescue #PWR013
+L Meow-Meow-rescue:GND-MeowMeow-Meow-Meow-rescue-Meow-Meow-rescue #PWR013
 U 1 1 5ADA141E
 P 9020 1630
@@
 $EndComp
 $Comp
-L Meow-Meow-rescue:GND-MeowMeow-Meow-Meow-rescue #PWR012
+L Meow-Meow-rescue:GND-MeowMeow-Meow-Meow-rescue-Meow-Meow-rescue #PWR012
 U 1 1 5ADA139A
 P 9255 1630
@@
 $EndComp
 $Comp
-L Meow-Meow-rescue:+3.3V-MeowMeow-Meow-Meow-rescue #PWR011
+L Meow-Meow-rescue:+3.3V-MeowMeow-Meow-Meow-rescue-Meow-Meow-rescue #PWR011
 U 1 1 5ADA11F4
 P 9595 1225
@@
 $EndComp
 $Comp
-L Meow-Meow-rescue:C_Small-MeowMeow-Meow-Meow-rescue C6
+L Meow-Meow-rescue:C_Small-MeowMeow-Meow-Meow-rescue-Meow-Meow-rescue C6
 U 1 1 5AD98F7F
 P 9255 1455
@@
 $EndComp
 $Comp
-L Meow-Meow-rescue:C_Small-MeowMeow-Meow-Meow-rescue C5
+L Meow-Meow-rescue:C_Small-MeowMeow-Meow-Meow-rescue-Meow-Meow-rescue C5
 U 1 1 5AD98EFB
 P 9020 1455
@@
 Text Label 1920 3615 2    50   ~ 0
 MISO
-Text Label 1915 3715 2    50   ~ 0
-CS
 Text Notes 3900 780  0    60   ~ 0
 MICROCONTROLLER SAMD21
@@
 	2440 940  2335 940
 $Comp
-L Meow-Meow-rescue:C_Small-MeowMeow-Meow-Meow-rescue C1
+L Meow-Meow-rescue:C_Small-MeowMeow-Meow-Meow-rescue-Meow-Meow-rescue C1
 U 1 1 5AFCC5C3
 P 2235 940
@@
 $EndComp
 $Comp
-L Meow-Meow-rescue:GND-MeowMeow-Meow-Meow-rescue #PWR015
+L Meow-Meow-rescue:GND-MeowMeow-Meow-Meow-rescue-Meow-Meow-rescue #PWR015
 U 1 1 5AFCC90C
 P 2080 940
@@
 Wire Wire Line
 	8980 3580 8870 3580
+NoConn ~ 4225 5995
+NoConn ~ 3530 2515
 $EndSCHEMATC

Commit message: New floorplant
Parts:
- removed J3: SWD, symbol Connector_Generic:Conn_01x04
- added J3: Conn_01x06, Connector:Tag-Connect_TC2030-IDC-NL_2x03_P1.27mm_Vertical, symbol Connector_Generic:Conn_01x06
- added U3: ATSAMD21G18A-M, Package_QFP:TQFP-48_7x7mm_P0.5mm, symbol MCU_Microchip_SAMD:ATSAMD21G18A-M
- C1, C2, C4, C5, C6: symbol Meow-Meow-rescue:C_Small-MeowMeow-Meow-Meow-rescue-Meow-Meow-rescue -> Meow-Meow-rescue:C_Small-MeowMeow-Meow-Meow-rescue-Meow-Meow-rescue-Meow-Meow-rescue
- D1, D2: symbol Meow-Meow-rescue:LED-MeowMeow-Meow-Meow-rescue-Meow-Meow-rescue -> Meow-Meow-rescue:LED-MeowMeow-Meow-Meow-rescue-Meow-Meow-rescue-Meow-Meow-rescue
- P1, P10, P11, P12, P2, P3, P5, P6, P7, P8: symbol Meow-Meow-rescue:CONN_01X01_FEMALE-MeowMeow-Meow-Meow-rescue-Meow-Meow-rescue -> Meow-Meow-rescue:CONN_01X01_FEMALE-MeowMeow-Meow-Meow-rescue-Meow-Meow-rescue-Meow-Meow-rescue
- P9: symbol Meow-Meow-rescue:USB_OTG-MeowMeow-Meow-Meow-rescue-Meow-Meow-rescue -> Meow-Meow-rescue:USB_OTG-MeowMeow-Meow-Meow-rescue-Meow-Meow-rescue-Meow-Meow-rescue
- R2, R3: symbol Meow-Meow-rescue:R_Small-MeowMeow-Meow-Meow-rescue-Meow-Meow-rescue -> Meow-Meow-rescue:R_Small-MeowMeow-Meow-Meow-rescue-Meow-Meow-rescue-Meow-Meow-rescue
- SW1: symbol Meow-Meow-rescue:SW_Push-MeowMeow-Meow-Meow-rescue-Meow-Meow-rescue -> Meow-Meow-rescue:SW_Push-MeowMeow-Meow-Meow-rescue-Meow-Meow-rescue-Meow-Meow-rescue
- U2: symbol Meow-Meow-rescue:AP2112K-3.3-Regulator_Linear-Meow-Meow-rescue-Meow-Meow-rescue -> Meow-Meow-rescue:AP2112K-3.3-Regulator_Linear-Meow-Meow-rescue-Meow-Meow-rescue-Meow-Meow-rescue
Connections:
- net +3V3: now also C2.1, U1.17 (VDDIO), U1.36 (VDDIO), U1.44 (VDDIN), U1.6 (VDDANA), J3.1 (Pin_1), U3.17 (VDDIO), U3.36 (VDDIO), U3.44 (VDDIN), U3.6 (VDDANA)
- net A0: now also U3.13 (PA08)
- net A1: now also U3.14 (PA09)
- net A2: now also U3.15 (PA10)
- net A3: now also U3.16 (PA11)
- net D+: now also U3.34 (PA25)
- net D-: now also U3.33 (PA24)
- net GND: now also J3.5 (Pin_5), U3.18 (GND), U3.35 (GND), U3.42 (GND), U3.5 (GNDANA)
- net GPIO05: now also U1.30 (PA21), U3.30 (PA21); no longer U1.23 (PA14)
- net GPIO06: now also U1.29 (PA20), U3.29 (PA20); no longer U1.24 (PA15)
- net GPIO08: now also U3.19 (PB10)
- net GPIO09: now also U1.26 (PA17), U3.26 (PA17); no longer U1.25 (PA16)
- net GPIO10: now also U1.25 (PA16), U3.25 (PA16); no longer U1.26 (PA17)
- net GPIO11: now also U1.24 (PA15), U3.24 (PA15); no longer U1.29 (PA20)
- net GPIO12: now also U1.20 (PB11), U3.20 (PB11); no longer U1.30 (PA21)
- net GPIO13: now also U1.23 (PA14), U3.23 (PA14); no longer U1.32 (PA23)
- net MISO: now also U3.31 (PA22)
- net MOSI: now also U3.27 (PA18)
- net RESET: now also J3.3 (Pin_3), U3.40 (~RESET)
- net RX: now also U3.22 (PA13)
- net SCK: now also U3.28 (PA19)
- net SCL: now also U3.2 (PA01)
- net SDA: now also U3.1 (PA00)
- net SWCLK: now also J3.4 (Pin_4), U3.45 (PA30)
- net SWDIO: now also J3.2 (Pin_2), U3.46 (PA31)
- net TX: now also U3.21 (PA12)
- net Y0: now also U3.3 (PA02)
- net Y1: now also U3.4 (PA03)
- net Y14: now also U3.7 (PB08)
- net Y15: now also U3.8 (PB09)
- net Y2: now also U3.9 (PA04)
- net Y3: now also U3.10 (PA05)
- net Y4: now also U3.11 (PA06)
- net Y5: now also U3.12 (PA07)
- net Y8: now also U3.47 (PB02)
- net Y9: now also U3.48 (PB03)
- net vddcore: now reaches C1.1, U1.43 (VDDCORE)
- net vddcore: now also U3.43 (VDDCORE)
- no-connect marks 10 -> 16
Other:
- moved on the sheet: SW1
