File: hardware/Meow Meow.kicad_sch (KiCad schematic)
At the start: 32 parts, among them J1 Conn_Left, J2 Conn_Right, J3 SWD, P1 SPACE, P10 A, P11 W, P12 KEY_UP_ARROW, P2 KEY_DOWN_ARROW, P3 KEY_RIGHT_ARROW, P4 USB_C_Plug_USB2.0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

Commit message: Fix pins capacitive
Connections:
- net A0: now also U1.9 (PA04), U3.9 (PA04); no longer U1.16 (PA11), U3.16 (PA11)
- net A1: now also U1.10 (PA05), U3.10 (PA05); no longer U1.15 (PA10), U3.15 (PA10)
- net A2: now also U1.47 (PB02), U3.47 (PB02); no longer U1.14 (PA09), U3.14 (PA09)
- net A3: now also U1.12 (PA07), U3.12 (PA07); no longer U1.13 (PA08), U3.13 (PA08)
- net GPIO08: now also U1.48 (PB03), U3.48 (PB03); no longer U1.19 (PB10), U3.19 (PB10)
- net GPIO11: now also U1.7 (PB08), U3.7 (PB08); no longer U1.20 (PB11), U3.20 (PB11)
- net Y2: now also U1.19 (PB10), U3.19 (PB10); no longer U1.9 (PA04), U3.9 (PA04)
- net Y3: now also U1.20 (PB11), U3.20 (PB11); no longer U1.10 (PA05), U3.10 (PA05)
- net Y8: now also U1.15 (PA10), U3.15 (PA10); no longer U1.47 (PB02), U3.47 (PB02)
- net Y9: now also U1.16 (PA11), U3.16 (PA11); no longer U1.48 (PB03), U3.48 (PB03)
- removed net Y14: P8.1, U1.7 (PB08), U3.7 (PB08)
- removed net Y5: P12.1, U1.12 (PA07), U3.12 (PA07)
- new net Y6: P12.1, U1.13 (PA08), U3.13 (PA08)
- new net Y7: P8.1, U1.14 (PA09), U3.14 (PA09)
Changed lines of the file:
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@@
   (no_connect (at 32.893 80.264))
   (no_connect (at 66.04 32.004))
-  (no_connect (at 32.893 85.217))
+  (no_connect (at 32.893 85.344))
   (no_connect (at 76.835 175.133))
   (wire (pts (xy 106.045 175.133) (xy 107.315 175.133))
@@
     (effects (font (size 1.27 1.27)) (justify right bottom))
   )
-  (label "GPIO08" (at 91.44 80.264 0)
+  (label "GPIO08" (at 91.186 70.104 0)
     (effects (font (size 1.27 1.27)) (justify left bottom))
   )
@@
     (effects (font (size 1.27 1.27)) (justify right bottom))
   )
-  (label "A1" (at 106.68 66.548 180)
+  (label "A1" (at 106.934 53.848 180)
     (effects (font (size 1.27 1.27)) (justify right bottom))
   )
@@
     (effects (font (size 1.524 1.524)) (justify right bottom))
   )
-  (label "Y8" (at 91.44 72.644 0)
-    (effects (font (size 1.27 1.27)) (justify left bottom))
-  )
-  (label "Y9" (at 91.186 70.104 0)
-    (effects (font (size 1.27 1.27)) (justify left bottom))
+  (label "Y8" (at 32.893 67.564 180)
+    (effects (font (size 1.27 1.27)) (justify right bottom))
+  )
+  (label "Y9" (at 32.893 70.104 180)
+    (effects (font (size 1.27 1.27)) (justify right bottom))
   )
   (label "VDDCORE" (at 63.5 27.686 270)
@@
     (effects (font (size 1.27 1.27)) (justify right bottom))
   )
-  (label "Y14" (at 203.454 151.6634 270)
+  (label "Y7" (at 203.454 151.6634 270)
     (effects (font (size 1.524 1.524)) (justify right bottom))
   )
@@
     (effects (font (size 1.27 1.27)) (justify right bottom))
   )
-  (label "GPIO11" (at 168.91 81.788 0)
-    (effects (font (size 1.27 1.27)) (justify left bottom))
-  )
-  (label "A3" (at 32.893 62.484 180)
+  (label "GPIO11" (at 168.656 74.168 0)
+    (effects (font (size 1.27 1.27)) (justify left bottom))
+  )
+  (label "A3" (at 32.766 59.944 180)
     (effects (font (size 1.27 1.27)) (justify right bottom))
   )
@@
     (effects (font (size 0.7 0.7)) (justify right bottom))
   )
-  (label "A3" (at 106.934 61.468 180)
+  (label "A3" (at 106.68 58.928 180)
     (effects (font (size 1.27 1.27)) (justify right bottom))
   )
@@
     (effects (font (size 0.7 0.7)) (justify right bottom))
   )
-  (label "Y5" (at 106.68 58.928 180)
+  (label "Y6" (at 106.934 61.468 180)
     (effects (font (size 1.27 1.27)) (justify right bottom))
   )
@@
     (effects (font (size 1.27 1.27)) (justify left bottom))
   )
-  (label "Y5" (at 225.044 152.5524 270)
+  (label "Y6" (at 225.044 152.5524 270)
     (effects (font (size 1.524 1.524)) (justify right bottom))
   )
@@
     (effects (font (size 1.524 1.524)) (justify right bottom))
   )
-  (label "Y9" (at 168.656 69.088 0)
-    (effects (font (size 1.27 1.27)) (justify left bottom))
+  (label "Y9" (at 106.68 69.088 180)
+    (effects (font (size 1.27 1.27)) (justify right bottom))
   )
   (label "Y4" (at 233.045 152.4254 270)
@@
     (effects (font (size 1.524 1.524)) (justify right bottom))
   )
-  (label "A0" (at 106.68 69.088 180)
-    (effects (font (size 1.27 1.27)) (justify right bottom))
-  )
-  (label "Y2" (at 106.934 51.308 180)
-    (effects (font (size 1.27 1.27)) (justify right bottom))
+  (label "A0" (at 106.934 51.308 180)
+    (effects (font (size 1.27 1.27)) (justify right bottom))
+  )
+  (label "Y2" (at 168.91 79.248 0)
+    (effects (font (size 1.27 1.27)) (justify left bottom))
   )
   (label "SWDIO" (at 106.934 112.268 180)
@@
     (effects (font (size 1.27 1.27)) (justify right bottom))
   )
-  (label "Y2" (at 32.766 52.324 180)
-    (effects (font (size 1.27 1.27)) (justify right bottom))
+  (label "Y2" (at 91.44 80.264 0)
+    (effects (font (size 1.27 1.27)) (justify left bottom))
   )
   (label "VDDANA" (at 130.81 29.21 270)
@@
     (effects (font (size 1.27 1.27)) (justify right bottom))
   )
-  (label "Y3" (at 32.766 54.864 180)
-    (effects (font (size 1.27 1.27)) (justify right bottom))
+  (label "Y3" (at 91.44 82.804 0)
+    (effects (font (size 1.27 1.27)) (justify left bottom))
   )
   (label "GPIO12" (at 107.315 162.433 0)
@@
     (effects (font (size 1.27 1.27)) (justify right bottom))
   )
-  (label "Y8" (at 168.91 71.628 0)
-    (effects (font (size 1.27 1.27)) (justify left bottom))
-  )
-  (label "A1" (at 32.893 67.564 180)
-    (effects (font (size 1.27 1.27)) (justify right bottom))
-  )
-  (label "Y14" (at 91.186 75.184 0)
-    (effects (font (size 1.27 1.27)) (justify left bottom))
-  )
-  (label "A2" (at 32.893 65.024 180)
-    (effects (font (size 1.27 1.27)) (justify right bottom))
-  )
-  (label "GPIO11" (at 91.44 82.804 0)
+  (label "Y8" (at 106.68 66.548 180)
+    (effects (font (size 1.27 1.27)) (justify right bottom))
+  )
+  (label "A1" (at 32.766 54.864 180)
+    (effects (font (size 1.27 1.27)) (justify right bottom))
+  )
+  (label "Y7" (at 32.893 65.024 180)
+    (effects (font (size 1.27 1.27)) (justify right bottom))
+  )
+  (label "A2" (at 91.44 72.644 0)
+    (effects (font (size 1.27 1.27)) (justify left bottom))
+  )
+  (label "GPIO11" (at 91.186 75.184 0)
     (effects (font (size 1.27 1.27)) (justify left bottom))
   )
@@
     (effects (font (size 1.27 1.27)) (justify right bottom))
   )
-  (label "Y14" (at 168.656 74.168 0)
-    (effects (font (size 1.27 1.27)) (justify left bottom))
-  )
-  (label "A0" (at 32.893 70.104 180)
+  (label "Y7" (at 106.68 64.008 180)
+    (effects (font (size 1.27 1.27)) (justify right bottom))
+  )
+  (label "A0" (at 32.766 52.324 180)
     (effects (font (size 1.27 1.27)) (justify right bottom))
   )
@@
     (effects (font (size 1.524 1.524)) (justify right bottom))
   )
-  (label "Y5" (at 32.766 59.944 180)
+  (label "Y6" (at 32.893 62.484 180)
     (effects (font (size 1.27 1.27)) (justify right bottom))
   )
@@
     (effects (font (size 1.27 1.27)) (justify right bottom))
   )
-  (label "Y3" (at 106.934 53.848 180)
-    (effects (font (size 1.27 1.27)) (justify right bottom))
+  (label "Y3" (at 168.91 81.788 0)
+    (effects (font (size 1.27 1.27)) (justify left bottom))
   )
   (label "MOSI" (at 32.893 87.884 180)
@@
     (effects (font (size 1.524 1.524)) (justify right bottom))
   )
-  (label "A2" (at 106.68 64.008 180)
-    (effects (font (size 1.27 1.27)) (justify right bottom))
+  (label "A2" (at 168.91 71.628 0)
+    (effects (font (size 1.27 1.27)) (justify left bottom))
   )
   (label "A2" (at 76.835 167.513 180)
@@
     (effects (font (size 1.27 1.27)) (justify left bottom))
   )
-  (label "GPIO08" (at 168.91 79.248 0)
-    (effects (font (size 1.27 1.27)) (justify left bottom))
-  )
+  (label "GPIO08" (at 168.656 69.088 0)
+    (effects (font (size 1.27 1.27)) (justify left bottom))
+  )

Commit message: update layout and fix pins 3.2v
Parts:
- J1: footprint Connector_PinSocket_2.54mm:PinSocket_1x16_P2.54mm_Vertical_SMD_Pin1Left -> Connector_PinSocket_2.54mm:PinSocket_1x16_P2.54mm_Vertical_SMD_Pin1Right
Connections:
- net A0: now also U1.47 (PB02), U3.47 (PB02); no longer U1.9 (PA04), U3.9 (PA04)
- net A1: now also U1.9 (PA04), U3.9 (PA04); no longer U1.10 (PA05), U3.10 (PA05)
- net A2: now also U1.10 (PA05), U3.10 (PA05); no longer U1.47 (PB02), U3.47 (PB02)
- net Y0: now also P11.1; no longer P7.1
- net Y1: now also P10.1; no longer P6.1
- net Y15: now also P7.1; no longer P1.1
- net Y2: now also P2.1; no longer P5.1
- net Y3: now also P12.1; no longer P3.1
- net Y4: now also P6.1; no longer P2.1
- net Y6: now also P8.1; no longer P12.1
- net Y7: now also P1.1; no longer P8.1
- net Y8: now also P5.1; no longer P11.1
- net Y9: now also P3.1; no longer P10.1
Changed lines of the file:
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@@
     (effects (font (size 1.27 1.27)) (justify right bottom))
   )
-  (label "Y8" (at 218.186 152.2984 270)
+  (label "Y8" (at 249.301 152.1714 270)
     (effects (font (size 1.524 1.524)) (justify right bottom))
   )
@@
     (effects (font (size 1.27 1.27)) (justify right bottom))
   )
-  (label "A1" (at 106.934 53.848 180)
+  (label "A1" (at 106.934 51.308 180)
     (effects (font (size 1.27 1.27)) (justify right bottom))
   )
@@
     (effects (font (size 1.27 1.27)) (justify left bottom))
   )
-  (label "Y3" (at 241.427 152.1714 270)
+  (label "Y3" (at 225.044 152.5524 270)
     (effects (font (size 1.524 1.524)) (justify right bottom))
   )
@@
     (effects (font (size 1.27 1.27)) (justify right bottom))
   )
-  (label "Y7" (at 203.454 151.6634 270)
+  (label "Y7" (at 195.707 151.4094 270)
     (effects (font (size 1.524 1.524)) (justify right bottom))
   )
@@
     (effects (font (size 1.27 1.27)) (justify left bottom))
   )
-  (label "Y6" (at 225.044 152.5524 270)
+  (label "Y6" (at 203.454 151.6634 270)
     (effects (font (size 1.524 1.524)) (justify right bottom))
   )
@@
     (effects (font (size 1.27 1.27)) (justify right bottom))
   )
-  (label "Y15" (at 195.707 151.4094 270)
+  (label "Y15" (at 265.557 152.2984 270)
     (effects (font (size 1.524 1.524)) (justify right bottom))
   )
@@
     (effects (font (size 1.27 1.27)) (justify right bottom))
   )
-  (label "Y4" (at 233.045 152.4254 270)
+  (label "Y4" (at 257.81 152.2984 270)
     (effects (font (size 1.524 1.524)) (justify right bottom))
   )
@@
     (effects (font (size 1.524 1.524)) (justify right bottom))
   )
-  (label "A0" (at 106.934 51.308 180)
-    (effects (font (size 1.27 1.27)) (justify right bottom))
+  (label "A0" (at 168.91 71.628 0)
+    (effects (font (size 1.27 1.27)) (justify left bottom))
   )
   (label "Y2" (at 168.91 79.248 0)
@@
     (effects (font (size 1.27 1.27)) (justify right bottom))
   )
-  (label "A1" (at 32.766 54.864 180)
+  (label "A1" (at 32.766 52.324 180)
     (effects (font (size 1.27 1.27)) (justify right bottom))
   )
@@
     (effects (font (size 1.27 1.27)) (justify right bottom))
   )
-  (label "A2" (at 91.44 72.644 0)
-    (effects (font (size 1.27 1.27)) (justify left bottom))
+  (label "A2" (at 32.766 54.864 180)
+    (effects (font (size 1.27 1.27)) (justify right bottom))
   )
   (label "GPIO11" (at 91.186 75.184 0)
@@
     (effects (font (size 1.27 1.27)) (justify right bottom))
   )
-  (label "Y2" (at 249.301 152.1714 270)
+  (label "Y2" (at 233.045 152.4254 270)
     (effects (font (size 1.524 1.524)) (justify right bottom))
   )
@@
     (effects (font (size 1.27 1.27)) (justify right bottom))
   )
-  (label "Y0" (at 265.557 152.2984 270)
+  (label "Y0" (at 218.186 152.2984 270)
     (effects (font (size 1.524 1.524)) (justify right bottom))
   )
@@
     (effects (font (size 1.27 1.27)) (justify right bottom))
   )
-  (label "A0" (at 32.766 52.324 180)
-    (effects (font (size 1.27 1.27)) (justify right bottom))
+  (label "A0" (at 91.44 72.644 0)
+    (effects (font (size 1.27 1.27)) (justify left bottom))
   )
   (label "SDA" (at 107.315 180.213 0)
@@
     (effects (font (size 1.27 1.27)) (justify right bottom))
   )
-  (label "Y9" (at 211.074 152.4254 270)
+  (label "Y9" (at 241.427 152.1714 270)
     (effects (font (size 1.524 1.524)) (justify right bottom))
   )
@@
     (effects (font (size 1.27 1.27)) (justify right bottom))
   )
-  (label "Y1" (at 257.81 152.2984 270)
-    (effects (font (size 1.524 1.524)) (justify right bottom))
-  )
-  (label "A2" (at 168.91 71.628 0)
-    (effects (font (size 1.27 1.27)) (justify left bottom))
+  (label "Y1" (at 211.074 152.4254 270)
+    (effects (font (size 1.524 1.524)) (justify right bottom))
+  )
+  (label "A2" (at 106.934 53.848 180)
+    (effects (font (size 1.27 1.27)) (justify right bottom))
   )
   (label "A2" (at 76.835 167.513 180)
@@
     (property "Reference" "J1" (id 0) (at 84.455 149.733 0))
     (property "Value" "Conn_Left" (id 1) (at 86.995 170.053 90))
-    (property "Footprint" "Connector_PinSocket_2.54mm:PinSocket_1x16_P2.54mm_Vertical_SMD_Pin1Left" (id 2) (at 84.455 170.053 0)
+    (property "Footprint" "Connector_PinSocket_2.54mm:PinSocket_1x16_P2.54mm_Vertical_SMD_Pin1Right" (id 2) (at 84.455 170.053 0)
       (effects (font (size 1.27 1.27)) hide)
     )
@@
     )
     (path "/00000000-0000-0000-0000-00005d4e7baf"
-      (reference "J1") (unit 1) (value "Conn_Left") (footprint "Connector_PinSocket_2.54mm:PinSocket_1x16_P2.54mm_Vertical_SMD_Pin1Left")
+      (reference "J1") (unit 1) (value "Conn_Left") (footprint "Connector_PinSocket_2.54mm:PinSocket_1x16_P2.54mm_Vertical_SMD_Pin1Right")
     )
     (path "/00000000-0000-0000-0000-00005d4e69e8"
